File: PCB/NomadKeyboard.kicad_pcb (KiCad board)
At the start: 2 copper layers, 12 x 20.6 mm, 115 parts, among them J1 4PIN, SW1 SW_PUSH_LED, SW10 SW_PUSH_LED, SW11 SW_PUSH_LED, SW12 SW_PUSH_LED, SW13 SW_PUSH_LED, SW14 SW_PUSH_LED, SW15 SW_PUSH_LED, SW16 SW_PUSH_LED, SW17 SW_PUSH_LED, SW18 SW_PUSH_LED, SW19 SW_PUSH_LED, SW2 SW_PUSH_LED, SW20 SW_PUSH_LED, SW21 SW_PUSH_LED, SW22 SW_PUSH_LED, SW23 SW_PUSH_LED, SW24 SW_PUSH_LED, SW25 SW_PUSH_LED, SW26 SW_PUSH_LED, SW27 SW_PUSH_LED, SW28 SW_PUSH_LED, SW29 SW_PUSH_LED, SW3 SW_PUSH_LED, SW30 SW_PUSH_LED, SW31 SW_PUSH_LED, SW32 SW_PUSH_LED, SW33 SW_PUSH_LED, SW34 SW_PUSH_LED, SW35 SW_PUSH_LED, SW36 SW_PUSH_LED, SW37 SW_PUSH_LED, SW38 SW_PUSH_LED, SW39 SW_PUSH_LED, SW4 SW_PUSH_LED, SW40 SW_PUSH_LED, SW41 SW_PUSH_LED, SW42 SW_PUSH_LED, SW43 SW_PUSH_LED, SW44 SW_PUSH_LED, SW45 SW_PUSH_LED, SW46 SW_PUSH_LED, SW47 SW_PUSH_LED, SW49 SW_PUSH_LED, SW5 SW_PUSH_LED, SW50 SW_PUSH_LED, SW51 SW_PUSH_LED, SW52 SW_PUSH_LED, SW53 SW_PUSH_LED, SW54 SW_PUSH_LED, SW6 SW_PUSH_LED, SW7 SW_PUSH_LED, SW8 SW_PUSH_LED, SW9 SW_PUSH_LED, U1 RP2040

Commit message: WIP
Parts:
- removed G*** (x2): LOGO, Nomad:Nomad_Logo_20
- removed J1: 4PIN, SofleChoc:MJ-4PP-9
- added D48: D, SofleChoc:crkbd-diode, F.Cu at (114.8, 56.1)
- added D55: SK6812MINI, SofleChoc:SK6812MiniE, F.Cu at (109.1, 51.2)
- added D56: D, SofleChoc:crkbd-diode, F.Cu at (78.8, 27.6)
- added SW48: SW_PUSH_LED, SofleChoc:Choc_Hotswap_SK6812MiniE, F.Cu at (84.8, 32.1)
- added U1: RP2040, mcu:rp2040-zero-smd, B.Cu at (105.3, 30.1)
- moved D1 12.0 mm to (78.8, 44.6)
- moved U1 5.22 mm to (105.3, 30.1)
- moved TH1 4.66 mm to (109.3, 65.1)
Connections:
- J_RGB1 pad 1: LED -> Net-(D55-DOUT)
- SW1 pad 1: VCC -> VDD
- SW10 pad 1: VCC -> VDD
- SW11 pad 1: VCC -> VDD
- SW12 pad 1: VCC -> VDD
- SW13 pad 1: VCC -> VDD
- SW14 pad 1: VCC -> VDD
- SW15 pad 1: VCC -> VDD
- SW16 pad 1: VCC -> VDD
- SW17 pad 1: VCC -> VDD
- SW18 pad 1: VCC -> VDD
- SW19 pad 1: VCC -> VDD
- SW2 pad 1: VCC -> VDD
- SW20 pad 1: VCC -> VDD
- SW21 pad 1: VCC -> VDD
- SW22 pad 1: VCC -> VDD
- SW23 pad 1: VCC -> VDD
- SW24 pad 1: VCC -> VDD
- SW25 pad 1: VCC -> VDD
- SW26 pad 1: VCC -> VDD
- SW27 pad 1: VCC -> VDD
- SW28 pad 1: VCC -> VDD
- SW29 pad 1: VCC -> VDD
- SW3 pad 1: VCC -> VDD
- SW30 pad 1: VCC -> VDD
- SW31 pad 1: VCC -> VDD
- SW32 pad 1: VCC -> VDD
- SW33 pad 1: VCC -> VDD
- SW34 pad 1: VCC -> VDD
- SW35 pad 1: VCC -> VDD
- SW36 pad 1: VCC -> VDD
- SW37 pad 1: VCC -> VDD
- SW38 pad 1: VCC -> VDD
- SW39 pad 1: VCC -> VDD
- SW4 pad 1: VCC -> VDD
- SW40 pad 1: VCC -> VDD
- SW41 pad 1: VCC -> VDD
- SW42 pad 1: VCC -> VDD
- SW43 pad 1: VCC -> VDD
- SW44 pad 1: VCC -> VDD
- SW45 pad 1: VCC -> VDD
- SW46 pad 1: VCC -> VDD
- SW47 pad 1: VCC -> VDD
- SW49 pad 1: VCC -> VDD
- SW5 pad 1: VCC -> VDD
- SW50 pad 1: VCC -> VDD
- SW51 pad 1: VCC -> VDD
- SW52 pad 1: VCC -> VDD
- SW53 pad 1: VCC -> VDD
- SW54 pad 1: VCC -> VDD
- SW6 pad 1: VCC -> VDD
- SW7 pad 1: VCC -> VDD
- SW8 pad 1: VCC -> VDD
- SW9 pad 1: VCC -> VDD
- U1 pad 1: unconnected-(U1-TX(PD3)-Pad1) -> VDD
- U1 pad 10: COL6 -> RX
- U1 pad 11: COL7 -> TX
- U1 pad 12: COL8 -> LED
- U1 pad 13: enc_i -> ROW5
- U1 pad 14: enc_d -> ROW6
- U1 pad 15: unconnected-(U1-D14(PB3)-Pad15) -> COL8
- U1 pad 16: ROW6 -> COL7
- U1 pad 17: ROW4 -> COL6
- U1 pad 18: ROW3 -> COL5
- U1 pad 19: ROW2 -> COL4
- U1 pad 20: ROW1 -> COL3
- U1 pad 21: ROW0 -> COL2
- U1 pad 22: DATA -> COL1
- U1 pad 23: LED -> COL0
- U1 pad 3: VCC -> unconnected-(U1-3v3-Pad3)
- U1 pad 4: COL0 -> unconnected-(U1-GP29-Pad4)
- U1 pad 5: COL1 -> ROW0
- U1 pad 6: COL2 -> ROW1
- U1 pad 7: COL3 -> ROW2
- U1 pad 8: COL4 -> ROW3
- U1 pad 9: COL5 -> ROW4
Routing:
- net LED: vias 0 -> 1
Other:
- board size 12 x 20.6 mm -> 131.5 x 112.8 mm

Commit message: WIP
Parts:
- removed D56: D, SofleChoc:crkbd-diode
- removed SW48: SW_PUSH_LED, SofleChoc:Choc_Hotswap_SK6812MiniE
Routing:
- net COL0: track 0.00 -> 320.7 mm, vias 0 -> 3
- net COL1: track 0.00 -> 258.3 mm, vias 0 -> 2
- net COL2: track 0.00 -> 236.5 mm, vias 0 -> 2
- net COL4: track 0.00 -> 197.6 mm, vias 0 -> 1
- net COL3: track 0.00 -> 195.3 mm, vias 0 -> 1
- net COL5: track 0.00 -> 130.4 mm, vias 0 -> 1
- net COL8: track 0.00 -> 108.3 mm, vias 0 -> 2
- net COL7: track 0.00 -> 88.9 mm, vias 0 -> 2
- net COL6: track 0.00 -> 81.0 mm, vias 0 -> 2
- net Net-(D55-DOUT): track 0.00 -> 36.3 mm, vias 0 -> 1
- net LED: track 0.00 -> 20.0 mm, vias 1 -> 2
- net Net-(D34-A): track 0.00 -> 12.4 mm
- net Net-(D48-K): track 0.00 -> 9.50 mm

Commit message: WIP
Parts:
- added D56: D, SofleChoc:crkbd-diode, F.Cu at (78.3, 44.6)
- added J1: 4PIN, SofleChoc:MJ-4PP-9, F.Cu at (82.7, 18.7)
- added SW48: SW_PUSH_LED, SofleChoc:Choc_Hotswap_SK6812MiniE, F.Cu at (84.8, 49.1)
- moved TH2 48.8 mm to (190.6, 42.4)
- moved TH1 24.4 mm to (127.6, 81.4)
- moved D1 20.0 mm to (78.8, 64.6)
- moved SW1 20.0 mm to (84.8, 69.1)
- moved D8 17.0 mm to (92.3, 81.6)
- moved SW15 17.0 mm to (84.8, 103.1)
- moved SW42 17.0 mm to (84.8, 120.1)
- moved SW8 17.0 mm to (84.8, 86.1)
- moved D38 16.5 mm to (91.3, 115.1)
- moved D15 16.1 mm to (90.8, 97.6)
- moved SW29 15.7 mm to (120.0, 125.5)
- moved D22 15.7 mm to (111.3, 140.0)
- moved SW22 15.7 mm to (103.5, 135.0)
- moved D29 15.7 mm to (127.8, 130.5)
- moved TH3 13.5 mm to (104.8, 117.1)
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Connections:
- SW35 pad 4: Net-(SW1B-DOUT) -> Net-(SW35B-DIN)
- SW36 pad 2: Net-(SW36B-DOUT) -> Net-(SW1B-DIN)
- SW37 pad 4: Net-(SW15B-DOUT) -> Net-(SW37B-DIN)
- SW38 pad 2: Net-(SW38B-DOUT) -> Net-(SW15B-DIN)
- SW42 pad 2: Net-(SW15B-DIN) -> Net-(SW42B-DOUT)
- SW42 pad 4: Net-(SW38B-DOUT) -> Net-(SW22B-DOUT)
- SW43 pad 4: Net-(SW22B-DOUT) -> Net-(SW42B-DOUT)
- SW8 pad 2: Net-(SW1B-DIN) -> Net-(SW37B-DIN)
- SW8 pad 4: Net-(SW36B-DOUT) -> Net-(SW15B-DOUT)
- U1 pad 14: ROW6 -> unconnected-(U1-GP9-Pad14) (x2)
Routing:
- net ROW5: track 0.00 -> 403.1 mm, vias 0 -> 2
- net ROW3: track 0.00 -> 304.3 mm, vias 0 -> 4
- net ROW4: track 0.00 -> 287.6 mm, vias 0 -> 4
- net ROW0: track 0.00 -> 248.7 mm, vias 0 -> 6
- net ROW2: track 0.00 -> 232.7 mm, vias 0 -> 3
- net ROW1: track 0.00 -> 201.7 mm, vias 0 -> 3
- net Net-(SW22B-DOUT): track 0.00 -> 32.3 mm
- net Net-(SW42B-DOUT): track 0.00 -> 14.1 mm
- net LED: track 20.0 -> 23.5 mm
- net COL5: track 130.4 -> 127.2 mm
- net COL1: track 258.3 -> 261.5 mm
- net COL2: track 236.5 -> 233.7 mm
- net COL7: track 88.9 -> 89.7 mm
- net COL3: track 195.3 -> 194.8 mm
Other:
- board size 131.5 x 112.8 mm -> 187 x 130.2 mm

Commit message: WIP
Parts:
- added J2: 4PIN, SofleChoc:MJ-4PP-9, F.Cu at (95.9, 66.2)
- J_RGB1: moved to B.Cu
Routing:
- net LED_slave: track 0.00 -> 23.7 mm
- net Net-(D55-DOUT): track 36.4 -> 36.8 mm, vias 1 -> 0

Commit message: WIP
Parts:
- added JP1: bridge_without_numpad, Jumper:SolderJumper-2_P1.3mm_Open_TrianglePad1.0x1.5mm, F.Cu at (99.1, 89.8)
- added J_RGB1: RGB jumper, Jumper:SolderJumper-3_P2.0mm_Open_TrianglePad1.0x1.5mm, F.Cu at (131.6, 42.4)
- moved TH1 56.3 mm to (75.8, 59.1)
- moved J_RGB1 53.1 mm to (131.6, 42.4), turned to 180 degrees
- moved TH4 41.3 mm to (194.1, 100.4)
- moved D48 13.6 mm to (103.6, 63.9), turned to 0 degrees
- moved D41 13.5 mm to (61.3, 63.9)
- moved D1 11.8 mm to (90.6, 63.9)
- moved D55 6.17 mm to (104.6, 55.4)
- moved J2 4.12 mm to (95.9, 70.4)
- moved D27 2.06 mm to (185.8, 98.6)
- moved D2 0.50 mm to (133.3, 47.6)
Routing:
- net VDD: track 0.00 -> 211.0 mm, vias 0 -> 2
- net COL8: track 108.7 -> 178.2 mm
- net COL6: track 80.5 -> 149.9 mm
- net COL7: track 89.7 -> 137.7 mm
- net Net-(SW52B-DOUT): track 0.00 -> 44.6 mm
- net Net-(SW50B-DOUT): track 0.00 -> 43.8 mm, vias 0 -> 2
- net Net-(SW13B-DOUT): track 0.00 -> 41.7 mm
- net led_bridge: track 0.00 -> 41.1 mm
- net Net-(SW26B-DOUT): track 0.00 -> 40.2 mm
- net Net-(SW10B-DIN): track 0.00 -> 39.9 mm
- net Net-(SW27B-DOUT): track 0.00 -> 39.9 mm
- net Net-(SW24B-DOUT): track 0.00 -> 39.9 mm
- net Net-(SW46B-DOUT): track 0.00 -> 39.4 mm
- net Net-(SW1B-DIN): track 0.00 -> 39.4 mm
- net Net-(SW38B-DIN): track 0.00 -> 39.3 mm
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Other:
- outline, holes or cut-outs redrawn
- board text added: "close when numpad is removed"
- board text added: "populate only"
- board text added: "when rgb master"
