File: PCB/NomadKeyboard.kicad_sch (KiCad schematic)
At the start: 90 parts, among them J1 4PIN, SW1 SW_PUSH_LED, SW10 SW_PUSH_LED, SW11 SW_PUSH_LED, SW12 SW_PUSH_LED, SW13 SW_PUSH_LED, SW14 SW_PUSH_LED, SW15 SW_PUSH_LED, SW16 SW_PUSH_LED, SW17 SW_PUSH_LED, SW18 SW_PUSH_LED, SW19 SW_PUSH_LED, SW2 SW_PUSH_LED, SW20 SW_PUSH_LED, SW21 SW_PUSH_LED, SW22 SW_PUSH_LED, SW23 SW_PUSH_LED, SW24 SW_PUSH_LED, SW25 SW_PUSH_LED, SW26 SW_PUSH_LED, SW27 SW_PUSH_LED, SW28 SW_PUSH_LED, SW29 SW_PUSH_LED, SW3 SW_PUSH_LED, SW30 SW_PUSH_LED, SW31 SW_PUSH_LED, SW32 SW_PUSH_LED, SW33 SW_PUSH_LED, SW34 SW_PUSH_LED, SW35 SW_PUSH_LED, SW36 SW_PUSH_LED, SW37 SW_PUSH_LED, SW38 SW_PUSH_LED, SW39 SW_PUSH_LED, SW4 SW_PUSH_LED, SW40 SW_PUSH_LED, SW41 SW_PUSH_LED, SW42 RotaryEncoder_Switch, SW5 SW_PUSH_LED, SW6 SW_PUSH_LED, SW7 SW_PUSH_LED, SW8 SW_PUSH_LED, SW9 SW_PUSH_LED, U1 RP2040

Commit message: row stagger layout
Parts:
- removed SW42: RotaryEncoder_Switch, Rotary_Encoder:RotaryEncoder_Alps_EC11E-Switch_Vertical_H20mm, symbol Device:RotaryEncoder_Switch
- added D38, D39, D44, D45, D46, D47, D49, D50, D51, D52, D53, D54: D, SofleChoc:crkbd-diode, symbol SofleKeyboard-rescue:D-Lily58-cache-Lily58_Pro-rescue
- added SW42, SW43, SW44, SW45, SW46, SW47, SW49, SW50, SW51, SW52, SW53, SW54: SW_PUSH_LED, SofleChoc:Choc_Hotswap_SK6812MiniE, symbol SofleKeyboard:SW_PUSH_LED
- U1: footprint RP2040:RP2040-mini -> mcu:rp2040-zero-smd
Connections:
- net COL0: now also SW54.6
- net COL1: now also SW53.6
- net COL2: now also SW52.6
- net COL3: now also SW51.6
- net COL4: now also SW50.6
- net COL5: now also SW29.6, SW49.6
- net COL6: now also SW42.6; no longer SW29.6
- net COL7: now also SW43.6, SW47.6
- net COL8: now also SW44.6, SW45.6, SW46.6
- net GND: now also SW42.3 (GND), SW43.3 (GND), SW44.3 (GND), SW45.3 (GND), SW46.3 (GND), SW47.3 (GND), SW49.3 (GND), SW50.3 (GND), SW51.3 (GND), SW52.3 (GND), SW53.3 (GND), SW54.3 (GND)
- net LED_start: now also SW49.4 (DIN); no longer SW41.4 (DIN)
- net ROW0: now also D46.1 (K), D47.1 (K), D49.1 (K), D50.1 (K), D51.1 (K), D52.1 (K), D53.1 (K), D54.1 (K); no longer D1.1 (K), D2.1 (K), D3.1 (K), D35.1 (K), D4.1 (K), D40.1 (K), D5.1 (K), D6.1 (K), D7.1 (K)
- net ROW1: now also D1.1 (K), D2.1 (K), D3.1 (K), D35.1 (K), D4.1 (K), D40.1 (K), D5.1 (K), D6.1 (K), D7.1 (K); no longer D10.1 (K), D11.1 (K), D12.1 (K), D13.1 (K), D14.1 (K), D36.1 (K), D41.1 (K), D8.1 (K), D9.1 (K)
- net ROW2: now also D10.1 (K), D11.1 (K), D12.1 (K), D13.1 (K), D14.1 (K), D36.1 (K), D41.1 (K), D8.1 (K), D9.1 (K); no longer D15.1 (K), D16.1 (K), D17.1 (K), D18.1 (K), D19.1 (K), D20.1 (K), D21.1 (K), D37.1 (K), D42.1 (K)
- net ROW3: now also D15.1 (K), D16.1 (K), D17.1 (K), D18.1 (K), D19.1 (K), D20.1 (K), D21.1 (K), D37.1 (K), D42.1 (K); no longer D22.1 (K), D23.1 (K), D24.1 (K), D25.1 (K), D26.1 (K), D27.1 (K), D28.1 (K), D43.1 (K)
- net ROW4: now also D23.1 (K), D24.1 (K), D25.1 (K), D26.1 (K), D27.1 (K), D28.1 (K), D43.1 (K), D38.1 (K), D44.1 (K); no longer D29.1 (K), D30.1 (K), D31.1 (K), D32.1 (K), D33.1 (K), D34.1 (K)
- net VCC: now also SW42.1 (VDD), SW43.1 (VDD), SW44.1 (VDD), SW45.1 (VDD), SW46.1 (VDD), SW47.1 (VDD), SW49.1 (VDD), SW50.1 (VDD), SW51.1 (VDD), SW52.1 (VDD), SW53.1 (VDD), SW54.1 (VDD)
- net led_bridge: now also SW47.2 (DOUT); no longer SW34.2 (DOUT)
- net at SW1.2 (DOUT): now also SW35.4 (DIN); no longer SW8.4 (DIN)
- net at SW1.4 (DIN): now also SW8.2 (DOUT); no longer SW35.2 (DOUT)
- net at SW3.2 (DOUT): now also SW2.4 (DIN); no longer SW10.4 (DIN)
- net at SW3.4 (DIN): now also SW4.2 (DOUT); no longer SW2.2 (DOUT)
- net at SW5.4 (DIN): now also SW6.2 (DOUT); no longer SW4.2 (DOUT)
- net at SW4.4 (DIN): now also SW5.2 (DOUT); no longer SW11.2 (DOUT)
- net at SW12.4 (DIN): now also SW11.2 (DOUT); no longer SW5.2 (DOUT)
- net at SW7.4 (DIN): now also SW54.2 (DOUT); no longer SW6.2 (DOUT)
- net at SW6.4 (DIN): now also SW7.2 (DOUT); no longer SW13.2 (DOUT)
- net at SW14.4 (DIN): now also SW13.2 (DOUT); no longer SW7.2 (DOUT)
- net at SW36.4 (DIN): now also SW40.2 (DOUT); no longer SW8.2 (DOUT)
- net at SW9.2 (DOUT): now also SW10.4 (DIN); no longer SW2.4 (DIN)
- net at SW11.4 (DIN): now also SW10.2 (DOUT); no longer SW18.2 (DOUT)
- net at SW12.2 (DOUT): now also SW13.4 (DIN); no longer SW19.4 (DIN)
- net at SW20.2 (DOUT): now also SW19.4 (DIN); no longer SW13.4 (DIN)
- net at SW28.4 (DIN): now also SW27.2 (DOUT); no longer SW21.2 (DOUT)
- net at SW20.4 (DIN): now also SW21.2 (DOUT); no longer SW27.2 (DOUT)
- net at SW27.4 (DIN): now also SW26.2 (DOUT); no longer SW33.2 (DOUT)
- net at SW32.4 (DIN): now also SW33.2 (DOUT); no longer SW26.2 (DOUT)
- net at SW26.4 (DIN): now also SW25.2 (DOUT); no longer SW19.2 (DOUT)
- net at SW18.4 (DIN): now also SW19.2 (DOUT); no longer SW25.2 (DOUT)
- net at SW25.4 (DIN): now also SW24.2 (DOUT); no longer SW31.2 (DOUT)
- net at SW9.4 (DIN): now also SW2.2 (DOUT); no longer SW16.2 (DOUT)
- net at SW16.4 (DIN): now also SW17.2 (DOUT); no longer SW23.2 (DOUT)
- net at SW23.4 (DIN): now also SW16.2 (DOUT); no longer SW29.2 (DOUT)
- net at SW29.4 (DIN): now also SW30.2 (DOUT); no longer SW22.2 (DOUT)
- net at SW15.2 (DOUT): now also SW37.4 (DIN); no longer SW38.4 (DIN)
- net at SW15.4 (DIN): now also SW42.2 (DOUT); no longer SW37.2 (DOUT)
- net at SW33.4 (DIN): now also SW34.2 (DOUT); no longer SW32.2 (DOUT)
- net at SW31.4 (DIN): now also SW32.2 (DOUT); no longer SW30.2 (DOUT)
- net at SW22.4 (DIN): now also SW29.2 (DOUT); no longer SW38.2 (DOUT)
- net at SW39.2 (DOUT): now also SW40.4 (DIN); no longer SW37.4 (DIN)
- net at SW39.4 (DIN): now also SW37.2 (DOUT); no longer SW40.2 (DOUT)
- net at SW36.2 (DOUT): now also SW8.4 (DIN); no longer SW40.4 (DIN)
- net at SW30.4 (DIN): now also SW31.2 (DOUT); no longer SW24.2 (DOUT)
- net at SW41.2 (DOUT): now also SW46.4 (DIN); no longer SW35.4 (DIN)
- net at SW17.4 (DIN): now also SW18.2 (DOUT); no longer SW10.2 (DOUT)
- net at SW24.4 (DIN): now also SW23.2 (DOUT); no longer SW17.2 (DOUT)
- net enc_s renamed ROW6
- new net: SW22.2 (DOUT), SW43.4 (DIN)
- new net: D53.2 (A), SW53.5
- new net: D52.2 (A), SW52.5
- new net: SW51.2 (DOUT), SW52.4 (DIN)
- new net: SW50.2 (DOUT), SW51.4 (DIN)
- new net: SW49.2 (DOUT), SW50.4 (DIN)
- new net: SW46.2 (DOUT), SW47.4 (DIN)
- new net: D44.2 (A), SW44.5
- new net: SW38.2 (DOUT), SW42.4 (DIN)
- new net: D46.2 (A), SW46.5
- new net: D49.2 (A), SW49.5
- new net: D51.2 (A), SW51.5
- new net: SW53.2 (DOUT), SW54.4 (DIN)
- new net: SW52.2 (DOUT), SW53.4 (DIN)
- new net: SW38.4 (DIN), SW44.2 (DOUT)
- new net: SW44.4 (DIN), SW45.2 (DOUT)
- new net: D54.2 (A), SW54.5
- new net: D45.2 (A), SW45.5
- new net: SW43.2 (DOUT), SW45.4 (DIN)
- new net: SW35.2 (DOUT), SW41.4 (DIN)
- new net: D47.2 (A), SW47.5
- new net: D50.2 (A), SW50.5
- new net: D39.2 (A), SW43.5
- new net: D38.2 (A), SW42.5
- new net ROW5: D22.1 (K), D29.1 (K), D30.1 (K), D31.1 (K), D32.1 (K), D33.1 (K), D34.1 (K), D39.1 (K), D45.1 (K)
Other:
- moved on the sheet: D1, D10, D11, D12, D13, D14, D15, D16, D17, D18, D19, D2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

Commit message: WIP
Parts:
- removed J1: 4PIN, SofleChoc:MJ-4PP-9, symbol SofleKeyboard-rescue:MJ-4PP-9-Lily58-cache-Lily58_Pro-rescue
- added D48: D, SofleChoc:crkbd-diode, symbol Device:D
- added D55: SK6812MINI, SofleChoc:SK6812MiniE, symbol LED:SK6812MINI
- added D56: D, SofleChoc:crkbd-diode, symbol SofleKeyboard-rescue:D-Lily58-cache-Lily58_Pro-rescue
- added SW48: SW_PUSH_LED, SofleChoc:Choc_Hotswap_SK6812MiniE, symbol SofleKeyboard:SW_PUSH_LED
Connections:
- net DATA is gone; now on net COL1: U1.22 (GP1(RX0))
- net enc_d is gone; now on net ROW6: U1.14 (GP9)
- net enc_i is gone; now on net ROW5: U1.13 (GP10)
- net COL0: now also U1.23 (GP0(TX0)); no longer U1.4 (GND)
- net COL1: no longer U1.5 (SDA(PD1))
- net COL2: now also U1.21 (GP2); no longer U1.6 (SCL(PD0))
- net COL3: now also U1.20 (GP3); no longer U1.7 (D4(PD4))
- net COL4: now also U1.19 (GP4); no longer U1.8 (D5(PC6))
- net COL5: now also U1.18 (GP5); no longer U1.9 (D6(PD7))
- net COL6: now also U1.17 (GP6), SW48.6; no longer U1.10 (D7(PE6))
- net COL7: now also U1.16 (GP7); no longer U1.11 (D8(PB4))
- net COL8: now also U1.15 (GP8); no longer U1.12 (D9(PB5))
- net GND: now also D55.2 (VSS)
- net LED: now also U1.12 (GP11), D55.3 (DIN); no longer J_RGB1.1 (A), U1.23 (GND)
- net ROW0: now also U1.5 (GP28), D56.1 (K); no longer U1.21 (VCC)
- net ROW1: now also U1.6 (GP27); no longer U1.20 (A3(PF4))
- net ROW2: now also U1.7 (GP26); no longer U1.19 (A2(PF5))
- net ROW3: now also U1.8 (GP15); no longer U1.18 (A1(PF6))
- net ROW4: now also U1.9 (GP14); no longer U1.17 (A0(PF7))
- net ROW6: no longer U1.16 (D15(PB1))
- net VCC: no longer SW1.1 (VDD), SW10.1 (VDD), SW11.1 (VDD), SW12.1 (VDD), SW13.1 (VDD), SW14.1 (VDD), SW15.1 (VDD), SW16.1 (VDD), SW17.1 (VDD), SW18.1 (VDD), SW19.1 (VDD), SW2.1 (VDD), SW20.1 (VDD), SW21.1 (VDD), SW22.1 (VDD), SW23.1 (VDD), SW24.1 (VDD), SW25.1 (VDD), SW26.1 (VDD), SW27.1 (VDD), SW28.1 (VDD), SW29.1 (VDD), SW3.1 (VDD), SW30.1 (VDD), SW31.1 (VDD), SW32.1 (VDD), SW33.1 (VDD), SW34.1 (VDD), SW35.1 (VDD), SW36.1 (VDD), SW37.1 (VDD), SW38.1 (VDD), SW39.1 (VDD), SW4.1 (VDD), SW40.1 (VDD), SW41.1 (VDD), SW42.1 (VDD), SW43.1 (VDD), SW44.1 (VDD), SW45.1 (VDD), SW46.1 (VDD), SW47.1 (VDD), SW49.1 (VDD), SW5.1 (VDD), SW50.1 (VDD), SW51.1 (VDD), SW52.1 (VDD), SW53.1 (VDD), SW54.1 (VDD), SW6.1 (VDD), SW7.1 (VDD), SW8.1 (VDD), SW9.1 (VDD), U1.3 (GND)
- net VDD: now reaches U1.1 (VDD)
- net VDD: now also SW1.1 (VDD), SW10.1 (VDD), SW11.1 (VDD), SW12.1 (VDD), SW13.1 (VDD), SW14.1 (VDD), SW15.1 (VDD), SW16.1 (VDD), SW17.1 (VDD), SW18.1 (VDD), SW19.1 (VDD), SW2.1 (VDD), SW20.1 (VDD), SW21.1 (VDD), SW22.1 (VDD), SW23.1 (VDD), SW24.1 (VDD), SW25.1 (VDD), SW26.1 (VDD), SW27.1 (VDD), SW28.1 (VDD), SW29.1 (VDD), SW3.1 (VDD), SW30.1 (VDD), SW31.1 (VDD), SW32.1 (VDD), SW33.1 (VDD), SW34.1 (VDD), SW35.1 (VDD), SW36.1 (VDD), SW37.1 (VDD), SW38.1 (VDD), SW39.1 (VDD), SW4.1 (VDD), SW40.1 (VDD), SW41.1 (VDD), SW42.1 (VDD), SW43.1 (VDD), SW44.1 (VDD), SW45.1 (VDD), SW46.1 (VDD), SW47.1 (VDD), SW49.1 (VDD), SW5.1 (VDD), SW50.1 (VDD), SW51.1 (VDD), SW52.1 (VDD), SW53.1 (VDD), SW54.1 (VDD), SW6.1 (VDD), SW7.1 (VDD), SW8.1 (VDD), SW9.1 (VDD), D48.2 (A)
- new net: D56.2 (A), SW48.5
- new net: D48.1 (K), D55.4 (VDD)
- new net: D55.1 (DOUT), J_RGB1.1 (A)
- new net RX: U1.10 (GP13(RX0))
- new net TX: U1.11 (GP12(TX0))
Other:
- moved on the sheet: J_RGB1

Commit message: WIP
Parts:
- removed D56: D, SofleChoc:crkbd-diode, symbol SofleKeyboard-rescue:D-Lily58-cache-Lily58_Pro-rescue
- removed SW48: SW_PUSH_LED, SofleChoc:Choc_Hotswap_SK6812MiniE, symbol SofleKeyboard:SW_PUSH_LED
Changed lines of the file:
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@@
 	)
 	(junction
-		(at 388.62 12.7)
-		(diameter 0)
-		(color 0 0 0 0)
-	)
-	(junction
 		(at 429.26 93.98)
 		(diameter 0)
@@
 	)
 	(junction
-		(at 373.38 5.08)
-		(diameter 0)
-		(color 0 0 0 0)
-	)
-	(junction
 		(at 414.02 53.34)
 		(diameter 0)
@@
 	(wire
 		(pts
-			(xy 373.38 2.54) (xy 373.38 5.08)
+			(xy 373.38 2.54) (xy 373.38 20.32)
 		)
 		(stroke
@@
 	(wire
 		(pts
-			(xy 388.62 12.7) (xy 408.94 12.7)
-		)
-		(stroke
-			(width 0)
-			(type default)
-		)
-	)
-	(wire
-		(pts
 			(xy 414.02 69.85) (xy 414.02 86.36)
 		)
@@
 	(wire
 		(pts
-			(xy 368.3 12.7) (xy 388.62 12.7)
+			(xy 368.3 12.7) (xy 408.94 12.7)
 		)
 		(stroke
@@
 	(wire
 		(pts
-			(xy 373.38 5.08) (xy 373.38 20.32)
-		)
-		(stroke
-			(width 0)
-			(type default)
-		)
-	)
-	(wire
-		(pts
 			(xy 170.18 52.07) (xy 170.18 49.53)
 		)
@@
 	(symbol
 		(lib_id "SofleKeyboard:SW_PUSH_LED")
-		(at 381 5.08 0)
-		(unit 1)
-		(exclude_from_sim no)
-		(in_bom yes)
-		(on_board yes)
-		(dnp no)
-		(property "Reference" "SW48"
-			(at 381 1.27 0)
-			(effects
-				(font
-					(size 1.27 1.27)
-				)
-			)
-		)
-		(property "Value" "SW_PUSH_LED"
-			(at 381 7.62 0)
-			(effects
-				(font
-					(size 1.27 1.27)
-				)
-				(hide yes)
-			)
-		)
-		(property "Footprint" "SofleChoc:Choc_Hotswap_SK6812MiniE"
-			(at 381 5.08 0)
-			(effects
-				(font
-					(size 1.27 1.27)
-				)
-				(hide yes)
-			)
-		)
-		(property "Datasheet" ""
-			(at 381 5.08 0)
-			(effects
-				(font
-					(size 1.27 1.27)
-				)
-				(hide yes)
-			)
-		)
-		(property "Description" ""
-			(at 381 5.08 0)
-			(effects
-				(font
-					(size 1.27 1.27)
-				)
-				(hide yes)
-			)
-		)
-		(pin "2"
-		)
-		(pin "3"
-		)
-		(pin "4"
-		)
-		(pin "6"
-		)
-		(pin "1"
-		)
-		(pin "5"
-		)
-		(instances
-			(project "NomadKeyboard"
-				(path "/eaee3b4b-85c3-461f-869e-93e0a5fc0df7"
-					(reference "SW48")
-					(unit 1)
-				)
-			)
-		)
-	)
-	(symbol
-		(lib_id "SofleKeyboard:SW_PUSH_LED")
 		(at 121.92 88.9 0)
 		(unit 2)
@@
 				)
 			)
-		)
-	)
-	(symbol
-		(lib_id "SofleKeyboard-rescue:D-Lily58-cache-Lily58_Pro-rescue")
-		(at 388.62 8.89 90)
-		(unit 1)
-		(exclude_from_sim no)
-		(in_bom yes)
-		(on_board yes)
-		(dnp no)
-		(property "Reference" "D56"
-			(at 384.302 7.366 90)
-			(effects
-				(font
-					(size 1.27 1.27)
-				)
-				(justify right)
-			)
-		)
-		(property "Value" "D"
-			(at 390.6266 10.033 90)
-			(effects
-				(font
-					(size 1.27 1.27)
-				)
-				(justify right)
-				(hide yes)
-			)
-		)
-		(property "Footprint" "SofleChoc:crkbd-diode"
-			(at 388.62 8.89 0)
-			(effects
-				(font
-					(size 1.27 1.27)
-				)
-				(hide yes)
-			)
-		)
-		(property "Datasheet" ""
-			(at 388.62 8.89 0)
-			(effects
-				(font
-					(size 1.27 1.27)
-				)
-				(hide yes)
-			)
-		)
-		(property "Description" ""
-			(at 388.62 8.89 0)
-			(effects
-				(font
-					(size 1.27 1.27)
-				)
-				(hide yes)
-			)
-		)
-		(pin "1"
-		)
-		(pin "2"
-		)
-		(instances
-			(project "NomadKeyboard"
-				(path "/eaee3b4b-85c3-461f-869e-93e0a5fc0df7"
-					(reference "D56")
-					(unit 1)
-				)
-			)

Commit message: WIP
Parts:
- added D56: D, SofleChoc:crkbd-diode, symbol SofleKeyboard-rescue:D-Lily58-cache-Lily58_Pro-rescue
- added J1, J2: 4PIN, SofleChoc:MJ-4PP-9, symbol SofleKeyboard-rescue:MJ-4PP-9-Lily58-cache-Lily58_Pro-rescue
- added SW48: SW_PUSH_LED, SofleChoc:Choc_Hotswap_SK6812MiniE, symbol SofleKeyboard:SW_PUSH_LED
Connections:
- net COL6: now also SW48.6
- net GND: now also J1.2, J2.2, SW48.3 (GND)
- net LED_slave: now also J1.5, J2.5
- net ROW0: now also D56.1 (K)
- net TX: now also J1.3, J2.3
- net VCC: now also J1.1, J2.1
- net VDD: now also SW48.1 (VDD)
- net led_bridge: now also J1.4, J2.4
- net at SW1.2 (DOUT): now also SW48.4 (DIN); no longer SW35.4 (DIN)
- net at SW1.4 (DIN): now also SW36.2 (DOUT); no longer SW8.2 (DOUT)
- net at SW8.4 (DIN): now also SW15.2 (DOUT); no longer SW36.2 (DOUT)
- net at SW37.4 (DIN): now also SW8.2 (DOUT); no longer SW15.2 (DOUT)
- net at SW15.4 (DIN): now also SW38.2 (DOUT); no longer SW42.2 (DOUT)
- net at SW22.2 (DOUT): now also SW42.4 (DIN); no longer SW43.4 (DIN)
- net ROW6: no longer names the net of U1.14 (GP9)
- new net: SW42.2 (DOUT), SW43.4 (DIN)
- new net: D56.2 (A), SW48.5
- new net: SW35.4 (DIN), SW48.2 (DOUT)
- no-connect marks 2 -> 3
Other:
- moved on the sheet: D48, D55, J_RGB1, SW15B, SW1B, SW22B, SW29B, SW35B, SW36B, SW42B, SW47B, SW8B

Commit message: WIP
Parts:
- added JP1: bridge_without_numpad, Jumper:SolderJumper-2_P1.3mm_Open_TrianglePad1.0x1.5mm, symbol Jumper:SolderJumper_2_Open
Connections:
- net led_bridge: now also JP1.2 (B)
- net at SW22.2 (DOUT), SW42.4 (DIN): now also JP1.1 (A)
Changed lines of the file:
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@@
 	)
 	(junction
+		(at 153.67 115.57)
+		(diameter 0)
+		(color 0 0 0 0)
+	)
+	(junction
 		(at 347.98 44.45)
 		(diameter 0)
@@
 	(wire
 		(pts
+			(xy 148.59 115.57) (xy 153.67 115.57)
+		)
+		(stroke
+			(width 0)
+			(type default)
+		)
+	)
+	(wire
+		(pts
 			(xy 170.18 63.5) (xy 170.18 60.96)
 		)
@@
 	(wire
 		(pts
+			(xy 148.59 128.27) (xy 148.59 115.57)
+		)
+		(stroke
+			(width 0)
+			(type default)
+		)
+	)
+	(wire
+		(pts
 			(xy 173.99 116.84) (xy 175.26 116.84)
 		)
@@
 		)
 	)
+	(global_label "led_bridge"
+		(shape input)
+		(at 140.97 128.27 180)
+		(fields_autoplaced yes)
+		(effects
+			(font
+				(size 1.27 1.27)
+			)
+			(justify right)
+		)
+		(property "Intersheetrefs" "${INTERSHEET_REFS}"
+			(at 128.842 128.27 0)
+			(effects
+				(font
+					(size 1.27 1.27)
+				)
+				(justify right)
+				(hide yes)
+			)
+		)
+	)
 	(global_label "ROW2"
 		(shape input)
@@
 				)
 			)
+		)
+	)
+	(symbol
+		(lib_id "Jumper:SolderJumper_2_Open")
+		(at 144.78 128.27 180)
+		(unit 1)
+		(exclude_from_sim yes)
+		(in_bom no)
+		(on_board yes)
+		(dnp no)
+		(fields_autoplaced yes)
+		(property "Reference" "JP1"
+			(at 144.78 121.92 0)
+			(effects
+				(font
+					(size 1.27 1.27)
+				)
+			)
+		)
+		(property "Value" "bridge_without_numpad"
+			(at 144.78 124.46 0)
+			(effects
+				(font
+					(size 1.27 1.27)
+				)
+			)
+		)
+		(property "Footprint" "Jumper:SolderJumper-2_P1.3mm_Open_TrianglePad1.0x1.5mm"
+			(at 144.78 128.27 0)
+			(effects
+				(font
+					(size 1.27 1.27)
+				)
+				(hide yes)
+			)
+		)
+		(property "Datasheet" "~"
+			(at 144.78 128.27 0)
+			(effects
+				(font
+					(size 1.27 1.27)
+				)
+				(hide yes)
+			)
+		)
+		(property "Description" "Solder Jumper, 2-pole, open"
+			(at 144.78 128.27 0)
+			(effects
+				(font
+					(size 1.27 1.27)
+				)
+				(hide yes)
+			)
+		)
+		(pin "2"
+		)
+		(pin "1"
+		)
+		(instances
+			(project ""
+				(path "/eaee3b4b-85c3-461f-869e-93e0a5fc0df7"
+					(reference "JP1")
+					(unit 1)
+				)
+			)

Commit message: WIP
Parts:
- added JP2: RightHand, Jumper:SolderJumper-2_P1.3mm_Open_TrianglePad1.0x1.5mm, symbol Jumper:SolderJumper_2_Open
Connections:
- net GND: now also JP2.2 (B)
- net VCC: no longer J1.1, J2.1
- net VDD: now also J1.1, J2.1
- net at U1.14 (GP9): now also JP2.1 (A)
- no-connect marks 3 -> 2
Changed lines of the file:
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@@
 		(at 27.94 26.67)
 	)
-	(no_connect
-		(at 60.96 46.99)
-	)
 	(wire
 		(pts
@@
 	(wire
 		(pts
+			(xy 60.96 46.99) (xy 73.66 46.99)
+		)
+		(stroke
+			(width 0)
+			(type default)
+		)
+	)
+	(wire
+		(pts
 			(xy 469.9 93.98) (xy 490.22 93.98)
 		)
@@
 			)
 		)
-		(property "Value" "VCC"
+		(property "Value" "VDD"
 			(at 62.6618 71.8058 0)
 			(effects
@@
 			)
 		)
-		(property "Value" "VCC"
+		(property "Value" "VDD"
 			(at 62.6618 98.4758 0)
 			(effects
@@
 	)
 	(symbol
+		(lib_id "SofleKeyboard-rescue:GND-Lily58-cache-Lily58_Pro-rescue")
+		(at 81.28 46.99 90)
+		(unit 1)
+		(exclude_from_sim no)
+		(in_bom yes)
+		(on_board yes)
+		(dnp no)
+		(property "Reference" "#PWR06"
+			(at 87.63 46.99 0)
+			(effects
+				(font
+					(size 1.27 1.27)
+				)
+				(hide yes)
+			)
+		)
+		(property "Value" "GND"
+			(at 85.09 46.99 0)
+			(effects
+				(font
+					(size 1.27 1.27)
+				)
+			)
+		)
+		(property "Footprint" ""
+			(at 81.28 46.99 0)
+			(effects
+				(font
+					(size 1.27 1.27)
+				)
+				(hide yes)
+			)
+		)
+		(property "Datasheet" ""
+			(at 81.28 46.99 0)
+			(effects
+				(font
+					(size 1.27 1.27)
+				)
+				(hide yes)
+			)
+		)
+		(property "Description" ""
+			(at 81.28 46.99 0)
+			(effects
+				(font
+					(size 1.27 1.27)
+				)
+				(hide yes)
+			)
+		)
+		(pin "1"
+		)
+		(instances
+			(project "NomadKeyboard"
+				(path "/eaee3b4b-85c3-461f-869e-93e0a5fc0df7"
+					(reference "#PWR06")
+					(unit 1)
+				)
+			)
+		)
+	)
+	(symbol
 		(lib_name "MJ-4PP-9-Lily58-cache-Lily58_Pro-rescue_1")
 		(lib_id "SofleKeyboard-rescue:MJ-4PP-9-Lily58-cache-Lily58_Pro-rescue")
@@
 					(unit 1)
 				)
+			)
+		)
+	)
+	(symbol
+		(lib_id "Jumper:SolderJumper_2_Open")
+		(at 77.47 46.99 0)
+		(unit 1)
+		(exclude_from_sim yes)
+		(in_bom no)
+		(on_board yes)
+		(dnp no)
+		(fields_autoplaced yes)
+		(property "Reference" "JP2"
+			(at 77.47 40.64 0)
+			(effects
+				(font
+					(size 1.27 1.27)
+				)
+			)
+		)
+		(property "Value" "RightHand"
+			(at 77.47 43.18 0)
+			(effects
+				(font
+					(size 1.27 1.27)
+				)
+			)
+		)
+		(property "Footprint" "Jumper:SolderJumper-2_P1.3mm_Open_TrianglePad1.0x1.5mm"
+			(at 77.47 46.99 0)
+			(effects
+				(font
+					(size 1.27 1.27)
+				)
+				(hide yes)
+			)
+		)
+		(property "Datasheet" "~"
+			(at 77.47 46.99 0)
+			(effects
+				(font
+					(size 1.27 1.27)
+				)
+				(hide yes)
+			)
+		)
+		(property "Description" "Solder Jumper, 2-pole, open"
+			(at 77.47 46.99 0)
+			(effects
+				(font
+					(size 1.27 1.27)
+				)
+				(hide yes)
+			)
+		)
+		(pin "2"
+		)
+		(pin "1"
+		)
+		(instances
+			(project ""
+				(path "/eaee3b4b-85c3-461f-869e-93e0a5fc0df7"
+					(reference "JP2")
+					(unit 1)
+				)

Commit message: after new layout
Parts:
- added JP3: LeftHand, Jumper:SolderJumper-2_P1.3mm_Open_TrianglePad1.0x1.5mm, symbol Jumper:SolderJumper_2_Open
Connections:
- net RX is gone; now on net COL5: U1.10 (GP13(RX0))
- net COL0: now also U1.5 (GP28); no longer U1.23 (GP0(TX0))
- net COL1: now also U1.6 (GP27); no longer U1.22 (GP1(RX0))
- net COL2: now also U1.7 (GP26); no longer U1.21 (GP2)
- net COL3: now also U1.8 (GP15); no longer U1.20 (GP3)
- net COL4: now also U1.9 (GP14); no longer U1.19 (GP4)
- net COL5: no longer U1.18 (GP5)
- net COL6: now also U1.21 (GP2); no longer U1.17 (GP6)
- net COL7: now also U1.22 (GP1(RX0)); no longer U1.16 (GP7)
- net COL8: now also U1.23 (GP0(TX0)); no longer U1.15 (GP8)
- net ROW0: now also U1.13 (GP10); no longer U1.5 (GP28)
- net ROW1: now also U1.14 (GP9); no longer U1.6 (GP27)
- net ROW2: now also U1.15 (GP8); no longer U1.7 (GP26)
- net ROW3: now also U1.16 (GP7); no longer U1.8 (GP15)
- net ROW4: now also U1.17 (GP6); no longer U1.9 (GP14)
- net ROW5: now also U1.18 (GP5); no longer U1.13 (GP10)
- net HAND: now reaches JP2.1 (A)
- net HAND: now also U1.4 (GP29), JP3.1 (A); no longer U1.14 (GP9)
- net 3v3: now reaches U1.3 (3v3)
- net 3v3: now also JP3.2 (B)
Other:
- moved on the sheet: JP2
